File: kicad/psu/psu/_autosave-psu.kicad_sch (KiCad schematic)
At the start: 17 parts, among them J1 AC, J2 DAC_PWR, J3 5V, U1 L7912, U2 uA7812

Commit message: WIP
Parts:
- J1: footprint (none) -> TerminalBlock_Phoenix:TerminalBlock_Phoenix_MPT-0,5-3-2.54_1x03_P2.54mm_Horizontal
Changed lines of the file:
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@@
 			)
 		)
-		(property "Footprint" ""
+		(property "Footprint" "TerminalBlock_Phoenix:TerminalBlock_Phoenix_MPT-0,5-3-2.54_1x03_P2.54mm_Horizontal"
 			(at 45.72 80.01 0)
 			(effects
