File: kicad/psu/psu/psu.kicad_pcb (KiCad board)
At the start: 2 copper layers, 93.5 x 38.5 mm, 21 parts, among them J1 AC, J2 DAC_PWR, J3 5V, U1 L7912, U2 uA7812

Commit message: WIP
Changed lines of the file:
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@@
 			(at 0 -4.15 0)
 			(layer "F.SilkS")
+			(hide yes)
 			(effects
 				(font

Commit message: WIP
Parts:
- removed U1: L7912, Package_TO_SOT_THT:TO-220-3_Vertical
- removed U2: uA7812, Package_TO_SOT_THT:TO-220-3_Vertical
- J2: value DAC_PWR -> Conn_01x03_Pin; footprint TerminalBlock_Phoenix:TerminalBlock_Phoenix_MPT-0,5-3-2.54_1x03_P2.54mm_Horizontal -> Connector_JST:JST_PH_B3B-PH-K_1x03_P2.00mm_Vertical
- J3: footprint TerminalBlock_Phoenix:TerminalBlock_Phoenix_MPT-0,5-2-2.54_1x02_P2.54mm_Horizontal -> Connector_JST:JST_PH_B2B-PH-K_1x02_P2.00mm_Vertical
- moved C6 11.0 mm to (143.8, 78.8), turned to -90 degrees
- moved C5 10.2 mm to (143.8, 69.1), turned to -90 degrees
- moved J2 7.76 mm to (150.6, 75.4), turned to -90 degrees
- moved J3 5.98 mm to (158.5, 84.6), turned to -90 degrees
- moved H2 3.80 mm to (164.2, 61.0)
- moved C7 3.45 mm to (157.6, 80.0)
- moved PS1 3.45 mm to (160.1, 71.0)
- moved H3 3.41 mm to (164.6, 92.2)
Connections:
- C1 pad 2: Net-(D1-A) -> -15V
- C2 pad 2: Net-(D1-A) -> -15V
- C3 pad 1: Net-(D3-K) -> +15V
- C4 pad 1: Net-(D3-K) -> +15V
- C5 pad 1: +12V -> +15V
- C6 pad 2: -12V -> -15V
- D1 pad 2: Net-(D1-A) -> -15V
- D2 pad 2: Net-(D1-A) -> -15V
- D3 pad 1: Net-(D3-K) -> +15V
- D4 pad 1: Net-(D3-K) -> +15V
- J2 pad 1: -12V -> +15V
- J2 pad 3: +12V -> -15V
- J3 pad 1: +5V -> GND
- J3 pad 2: GND -> +5V
- PS1 pad 1: +12V -> +15V
Routing:
- net +15V: track 0.00 -> 83.9 mm
- net Net-(D1-A): track 76.0 -> 0.00 mm
- net -15V: track 0.00 -> 69.6 mm
- net Net-(D3-K): track 68.5 -> 0.00 mm
- net +12V: track 30.4 -> 0.00 mm
- net -12V: track 13.3 -> 0.00 mm
- net +5V: track 16.0 -> 14.6 mm
Other:
- board size 93.5 x 38.5 mm -> 90.9 x 38.5 mm
- board text added: "+15V"
- board text added: "-15V"
- board text removed: "+12V"
- board text removed: "-12V"
