File: kicad/psu/psu/psu.kicad_sch (KiCad schematic)
At the start: 17 parts, among them J1 AC, J2 DAC_PWR, J3 5V, U1 L7912, U2 uA7812

Commit message: WIP
Parts:
- added H1, H2, H3, H4: MountingHole, MountingHole:MountingHole_3.2mm_M3, symbol Mechanical:MountingHole
- J1: footprint (none) -> TerminalBlock_Phoenix:TerminalBlock_Phoenix_MPT-0,5-3-2.54_1x03_P2.54mm_Horizontal

Commit message: WIP
Parts:
- removed J2: DAC_PWR, TerminalBlock_Phoenix:TerminalBlock_Phoenix_MPT-0,5-3-2.54_1x03_P2.54mm_Horizontal, symbol Connector:Screw_Terminal_01x03
- removed J3: 5V, TerminalBlock_Phoenix:TerminalBlock_Phoenix_MPT-0,5-2-2.54_1x02_P2.54mm_Horizontal, symbol Connector:Screw_Terminal_01x02
- removed U1: L7912, Package_TO_SOT_THT:TO-220-3_Vertical, symbol Regulator_Linear:L7912
- removed U2: uA7812, Package_TO_SOT_THT:TO-220-3_Vertical, symbol Regulator_Linear:uA7812
- added J2: Conn_01x03_Pin, Connector_JST:JST_PH_B3B-PH-K_1x03_P2.00mm_Vertical, symbol Connector:Conn_01x03_Pin
- added J3: 5V, Connector_JST:JST_PH_B2B-PH-K_1x02_P2.00mm_Vertical, symbol Connector:Conn_01x02_Pin
Connections:
- net +12V is gone; now on net +15V: C5.1, PS1.1 (+VIN)
- net -12V is gone; now on net -15V: C6.2
- net +5V: now also J3.2 (Pin_2)
- net GND: now also J2.2 (Pin_2), J3.1 (Pin_1)
- net +15V: now reaches C3.1, C4.1, D3.1 (K), D4.1 (K)
- net +15V: now also J2.1 (Pin_1)
- net -15V: now reaches C1.2, C2.2, D1.2 (A), D2.2 (A)
- net -15V: now also J2.3 (Pin_3)
Other:
- moved on the sheet: C1, C2, C3, C4, D1, D2, D3, D4, H1, H4, J1
