File: kicad/dac/dac.kicad_pcb (KiCad board)
At the start: 4 copper layers, 41.2 x 36 mm, 52 parts, among them U1 ES9039Q2M, U2 OPA1612AxD, U3 OPA1612AxD, U4 LT3046ATC+

Commit message: WIP
Parts:
- moved C21 54.0 mm to (140.2, 120.8)
- moved C17 53.3 mm to (135.5, 125.2)
- moved R18 52.5 mm to (123.3, 124.2)
- moved R17 52.3 mm to (117.8, 125.0)
- moved R15 41.1 mm to (126.2, 104.2), turned to 90 degrees
- moved R13 34.2 mm to (110.0, 110.5)
- moved R14 33.6 mm to (110.0, 112.2)
- moved C3 30.2 mm to (115.5, 92.0)
- moved C14 30.1 mm to (111.7, 120.8)
- moved R24 23.5 mm to (141.3, 125.2)
- moved R25 15.8 mm to (132.5, 112.8)
- moved R11 14.4 mm to (117.5, 101.2)
- moved C26 14.3 mm to (142.5, 102.0), turned to 90 degrees
- moved R12 14.3 mm to (112.0, 104.2)
- moved R20 14.1 mm to (139.5, 101.5)
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Routing:
- net DAC1B: track 23.2 -> 46.2 mm
- net DAC2: track 47.5 -> 37.4 mm
- net DAC2B: track 39.1 -> 30.3 mm, vias 4 -> 1
- net Net-(U3A--): track 16.3 -> 11.7 mm
- net Net-(C10-Pad2): track 12.9 -> 17.0 mm
- net Net-(C16-Pad2): track 29.7 -> 27.1 mm, vias 2 -> 4
- net Net-(C12-Pad2): track 25.8 -> 28.4 mm, vias 0 -> 2
- net DAC1: track 40.3 -> 42.7 mm
- net Net-(U2A--): track 13.4 -> 14.5 mm, vias 2 -> 4
- net Net-(C20-Pad1): track 19.3 -> 18.4 mm, vias 4 -> 0
- net GND: vias 34 -> 19
Other:
- board size 41.2 x 36 mm -> 45.5 x 36 mm
