File: kicad/dac/_autosave-dac.kicad_pcb (KiCad board)
At the start: 4 copper layers, 69.8 x 45 mm, 52 parts, among them U1 ES9039Q2M, U2 OPA1612AxD, U3 OPA1612AxD, U4 LT3046ATC+

Commit message: WIP
Parts:
- moved C24 42.8 mm to (126.8, 111.5), turned to 0 degrees
- moved C23 41.3 mm to (118.2, 105.5), turned to 0 degrees
- turned C13 to 180 degrees
- turned R16 to 180 degrees
- turned R18 to 180 degrees
Routing:
- net Net-(C12-Pad2): track 13.5 -> 34.4 mm
- net Net-(C10-Pad2): track 17.0 -> 35.3 mm
- net DAC1B: track 17.2 -> 35.1 mm, vias 0 -> 2
- net Net-(U2A--): track 7.33 -> 18.0 mm
- net DAC1: track 21.9 -> 29.1 mm
- net Net-(C15-Pad2): track 0.00 -> 1.59 mm
- net Net-(C14-Pad2): track 0.00 -> 1.56 mm
- removed copper zone on B.Cu, net GND
- removed copper zone on F.Cu, net GND
- removed copper zone on In1.Cu, net GND
