File: kicad/dac/dac.kicad_sch (KiCad schematic)
At the start: 23 parts, among them J1 I2S, J2 I2S, J3 ANALOG PWR, J4 5V, U1 ES9039Q2M, U4 LT3046ATC+, Y1 CE33xx

Commit message: WIP
Parts:
- removed C1, C2, C6: 4.7u, symbol Device:C_Polarized
- removed C8: 1u, symbol Device:C_Polarized
- removed J3: ANALOG PWR, symbol Connector:Screw_Terminal_01x03
- removed J4: 5V, symbol Connector:Screw_Terminal_01x02
- added C1, C2, C6, C8: 10u, Capacitor_SMD:C_0805_2012Metric, symbol Device:C
- added C28, C31: 10n, Capacitor_SMD:C_0603_1608Metric, symbol Device:C
- added C29, C30: 22u, Capacitor_Tantalum_SMD:CP_EIA-3216-10_Kemet-I_HandSolder, symbol Device:C_Polarized
- added C32: 100n, Capacitor_SMD:C_0402_1005Metric, symbol Device:C
- added H1: MountingHole, MountingHole:MountingHole_3.2mm_M3, symbol Mechanical:MountingHole
- added H2, H3, H4: MountingHole, symbol Mechanical:MountingHole
- added J3: ANALOG PWR, Connector_JST:JST_PH_B3B-PH-K_1x03_P2.00mm_Vertical, symbol Connector:Conn_01x03_Pin
- added J4: 5V, Connector_JST:JST_PH_B2B-PH-K_1x02_P2.00mm_Vertical, symbol Connector:Conn_01x02_Pin
- added R1: 90.9k, Resistor_SMD:R_0603_1608Metric_Pad0.98x0.95mm_HandSolder, symbol Device:R
- added R27, R3: 10k, Resistor_SMD:R_0603_1608Metric_Pad0.98x0.95mm_HandSolder, symbol Device:R
- added R28, R29, R30, R31, R32: 0, Resistor_SMD:R_0603_1608Metric_Pad0.98x0.95mm_HandSolder, symbol Device:R
- added R4: 100k, Resistor_SMD:R_0603_1608Metric_Pad0.98x0.95mm_HandSolder, symbol Device:R
- added U5: TPS7A39, Package_SON:Texas_S-PVSON-N10_ThermalVias, symbol Regulator_Linear:TPS7A39
- C27: footprint (none) -> Capacitor_Tantalum_SMD:CP_EIA-3216-10_Kemet-I_HandSolder; Vendor (none) -> Kyocera
- C3, C7: footprint Capacitor_SMD:C_0603_1608Metric -> Capacitor_SMD:C_0402_1005Metric; Vendor (none) -> Murata
- C4: value 100n -> 10n; Vendor (none) -> Kyocera
- C5: Vendor (none) -> Kyocera
- J1: footprint (none) -> Connector_JST:JST_PH_B3B-PH-K_1x03_P2.00mm_Vertical; Vendor (none) -> Amazon
- J2: footprint (none) -> Connector_JST:JST_PH_B4B-PH-K_1x04_P2.00mm_Vertical; Vendor (none) -> Amazon
- R10: value 100k -> 47k; Vendor (none) -> Panasonic
- R2: Vendor (none) -> Yaego
- R8, R9: value 50 -> 4.7k; Vendor (none) -> Panasonic; now left out of the parts list
- U1: footprint Package_DFN_QFN:UQFN-32_5x5mm_P0.5mm -> Package_DFN_QFN:UFQFPN-32-1EP_5x5mm_P0.5mm_EP3.5x3.5mm; Vendor (none) -> ESS
- U4: Vendor (none) -> TI
- Y1: value CE33xx -> CE3391-49.152; footprint SIT8209AI-G1-25E-156.253906Y:OSC_SIT8209AI-G1-25E-156.253906Y -> Oscillator:Oscillator_SMD_Diodes_FN-4Pin_7.0x5.0mm; Vendor (none) -> Crystek
Connections:
- net +12V: now also C4.1, C29.1, R1.1, R29.1, U5.10 (OUTP)
- net +3.3V: now also R8.1, R9.1, C2.1, C32.1, R28.1, R32.1; no longer C4.2
- net +5V: now also U4.7 (PGFB), C1.1, J4.2 (Pin_2), R29.2
- net -12V: now also C28.2, C30.2, R4.2, U5.6 (OUTN)
- net BCLK: now also J2.1 (Pin_1); no longer J2.2 (Pin_2)
- net DATA: now also J2.3 (Pin_3); no longer J2.4 (Pin_4)
- net GND: now also J2.4 (Pin_4), U1.33 (PAD), C1.2, C2.2, C29.2, C30.1, C31.2, C32.2, C6.2, C8.2, J3.2 (Pin_2), J4.1 (Pin_1), R3.1, R30.2, R31.2, U5.11 (GND), U5.4 (GND); no longer C4.1, J2.1 (Pin_1), U1.19 (ADDR1), U1.20 (ADDR0)
- net SCA: now also R8.2, U1.16 (SCA); no longer R9.2
- net SCL: now also R9.2, U1.15 (SCL); no longer R8.2
- net WCLK: now also J2.2 (Pin_2); no longer J2.3 (Pin_3)
- net at R10.2, U1.18 (CHIP_EN): now also C8.1
- net at U1.9 (DVDD): now also C6.1
- new net: C28.1, R27.1, R4.1, U5.7 (FBN)
- new net: R31.1, R32.2, U1.19 (ADDR1)
- new net: R28.2, R30.1, U1.20 (ADDR0)
- new net: R27.2, U5.8 (BUF)
- new net: C4.2, R1.2, R3.2, U5.9 (FBP)
- new net: C31.1, U5.3 (NR/SS)
- new net +15V: J3.1 (Pin_1), U5.1 (INP), U5.2 (EN)
- new net -15V: J3.3 (Pin_3), U5.5 (INN)
- no-connect marks 0 -> 10
Other:
- moved on the sheet: C27, C3, C7, J1, J2, R10, R2, R5, R6, R7, R8, R9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
