File: kicad/dac/output.kicad_sch (KiCad schematic)
At the start: 36 parts, among them U2 OPA1612AxD, U3 OPA1612AxD

Commit message: WIP
Parts:
- added J5: AUDIO OUT, Custom:SWITCHCRAFT_PJRAN2X1U01AUX, symbol Custom:PJRAN2X1U01AUX
- C10, C16, C22, C9: Vendor (none) -> Murata
- C11, C13, C19, C20: now left out of the parts list
- C12, C14, C15, C17, C18, C21: Vendor (none) -> Walsin
- C23, C24, C25, C26: Vendor (none) -> Kyocera
- R11, R12, R13, R14, R19, R20, R25, R26: Vendor (none) -> Yaego
- R15, R16, R22, R23: Vendor (none) -> Panasonic; now left out of the parts list
- R17, R18, R21, R24: Vendor (none) -> Vishay
- U2, U3: Vendor (none) -> TI
Connections:
- net GND: now also J5.1_A, J5.1_B
- net at C21.2, R24.2: now also J5.2_B, J5.3_B
- net at C15.2, R18.2: now also J5.2_A, J5.3_A
Other:
- moved on the sheet: C10, C15, C21, C22, R13, R14, R25, R26
