File: kicad/param-eq/param-eq.kicad_sch (KiCad schematic)
At the start: 1 part, among them U1 Teensy4.1

Commit message: WIP
Parts:
- added C1: 100n, Custom:C_Rect_L7.2mm_W3.0mm_P5.00mm_FKS2_FKP2_MKS2_MKP2_HandSolder, symbol Device:C
- added C2: 100u, Capacitor_THT:CP_Radial_D8.0mm_P5.00mm, symbol Device:C_Polarized
- added D1: SB140, Diode_THT:D_DO-41_SOD81_P10.16mm_Horizontal, symbol Diode:SB140
- added D2: 1N5233, Diode_THT:D_DO-41_SOD81_P10.16mm_Horizontal, symbol Diode:1N47xxA
- added H1, H2, H3, H4: MountingHole, MountingHole:MountingHole_3.2mm_M3, symbol Mechanical:MountingHole
- added J1: POWER, TerminalBlock_4Ucon:TerminalBlock_4Ucon_1x02_P3.50mm_Horizontal, symbol Connector:Screw_Terminal_01x02
- added J10: Q, Connector_JST:JST_PH_B4B-PH-K_1x04_P2.00mm_Vertical, symbol Connector:Conn_01x04_Pin
- added J11: GPIO, Connector_PinHeader_2.54mm:PinHeader_1x09_P2.54mm_Vertical, symbol Connector:Conn_01x09_Pin
- added J12: GAIN, Connector_JST:JST_PH_B4B-PH-K_1x04_P2.00mm_Vertical, symbol Connector:Conn_01x04_Pin
- added J13: FC, Connector_JST:JST_PH_B4B-PH-K_1x04_P2.00mm_Vertical, symbol Connector:Conn_01x04_Pin
- added J2, J4: I2S_IN, Connector_JST:JST_PH_B4B-PH-K_1x04_P2.00mm_Vertical, symbol Connector:Conn_01x04_Pin
- added J3: MGAIN, Connector_JST:JST_PH_B4B-PH-K_1x04_P2.00mm_Vertical, symbol Connector:Conn_01x04_Pin
- added J5: DISPLAY, Connector_JST:JST_PH_B3B-PH-K_1x03_P2.00mm_Vertical, symbol Connector:Conn_01x03_Pin
- added J6: DAC_CONTROL, Connector_JST:JST_PH_B3B-PH-K_1x03_P2.00mm_Vertical, symbol Connector:Conn_01x03_Pin
- added J7: S/PDIF, TestPoint:TestPoint_2Pads_Pitch2.54mm_Drill0.8mm, symbol Connector:Conn_Coaxial
- added J8: SPARE, Connector_JST:JST_PH_B4B-PH-K_1x04_P2.00mm_Vertical, symbol Connector:Conn_01x04_Pin
- added J9: CLIP_LED, Connector_JST:JST_PH_B2B-PH-K_1x02_P2.00mm_Vertical, symbol Connector:Conn_01x02_Pin
- added R1, R2, R3, R4, R5, R9: 100, Resistor_THT:R_Axial_DIN0204_L3.6mm_D1.6mm_P2.54mm_Vertical, symbol Device:R
- added R10: 75, Custom:R_Axial_DIN0204_L3.6mm_D1.6mm_P7.62mm_Horizontal_HandSolder, symbol Device:R
- added R11, R12, R13, R15, R16, R17, R18, R19, R20, R21, R22, R23, R6, R7, R8: 4.7k, Custom:R_Axial_DIN0204_L3.6mm_D1.6mm_P7.62mm_Horizontal_HandSolder, symbol Device:R
- added R14: 180, Custom:R_Axial_DIN0204_L3.6mm_D1.6mm_P7.62mm_Horizontal_HandSolder, symbol Device:R
- U1: footprint (none) -> Custom:Teensy41
Connections:
- net GND: now reaches U1.1 (GND)
- net GND: now also U1.34 (GND), U1.47 (GND), C1.2, C2.2, D2.2 (A), J1.2 (Pin_2), J10.4 (Pin_4), J11.1 (Pin_1), J12.4 (Pin_4), J13.4 (Pin_4), J2.4 (Pin_4), J3.1 (Pin_1), J4.4 (Pin_4), J5.1 (Pin_1), J6.1 (Pin_1), J7.2 (Ext), J8.1 (Pin_1), J9.1 (Pin_1), R10.2
- net SPBTN: now reaches U1.12 (10_CS_MQSR)
- net SPBTN: now also J8.2 (Pin_2), R13.2
- net SP_A: now reaches U1.13 (11_MOSI_CTX1)
- net SP_A: now also J8.3 (Pin_3), R12.2
- net SP_B: now reaches U1.14 (12_MISO_MQSL)
- net SP_B: now also J8.4 (Pin_4), R11.2
- net +3.3V: now reaches U1.15 (3V3)
- net +3.3V: now also R11.1, R12.1, R13.1, R15.2, R16.2, R17.2, R18.2, R19.2, R20.2, R21.2, R22.2, R23.2, R6.2, R7.2, R8.2
- net GPIO1: now reaches U1.17 (25_A11_RX6_SDA2)
- net GPIO1: now also J11.2 (Pin_2)
- net GPIO2: now reaches U1.18 (26_A12_MOSI1)
- net GPIO2: now also J11.3 (Pin_3)
- net GPIO3: now reaches U1.19 (27_A13_SCK1)
- net GPIO3: now also J11.4 (Pin_4)
- net GPIO4: now reaches U1.20 (28_RX7)
- net GPIO4: now also J11.5 (Pin_5)
- net GPIO5: now reaches U1.21 (29_TX7)
- net GPIO5: now also J11.6 (Pin_6)
- net GPIO6: now reaches U1.22 (30_CRX3)
- net GPIO6: now also J11.7 (Pin_7)
- net GPIO7: now reaches U1.23 (31_CTX3)
- net GPIO7: now also J11.8 (Pin_8)
- net GPIO8: now reaches U1.24 (32_OUT1B)
- net GPIO8: now also J11.9 (Pin_9)
- net FC_B: now reaches U1.25 (33_MCLK2)
- net FC_B: now also J13.1 (Pin_1), R15.1
- net FC_A: now reaches U1.26 (34_RX8)
- net FC_A: now also J13.2 (Pin_2), R20.1
- net FCBTN: now reaches U1.27 (35_TX8)
- net FCBTN: now also J13.3 (Pin_3), R16.1
- net FG: now reaches U1.28 (36_CS)
- net FG: now also J12.1 (Pin_1), R21.1
- net FG_A: now reaches U1.29 (37_CS)
- net FG_A: now also J12.2 (Pin_2), R17.1
- net MGBTN: now reaches U1.3 (1_TX1_CTX2_MISO1)
- net MGBTN: now also J3.2 (Pin_2), R6.1
- net FGBTN: now reaches U1.30 (38_CS1_IN1)
- net FGBTN: now also J12.3 (Pin_3), R22.1
- net Q_B: now reaches U1.31 (39_MISO1_OUT1A)
- net Q_B: now also J10.1 (Pin_1), R18.1
- net Q_A: now reaches U1.32 (40_A16)
- net Q_A: now also J10.2 (Pin_2), R23.1
- net QBTN: now reaches U1.33 (41_A17)
- net QBTN: now also J10.3 (Pin_3), R19.1
- net at U1.35 (13_SCK_LED): now also R14.1
- net at U1.37 (15_A1_RX3_SPDIF_IN): now also J7.1 (In), R10.1
- net MG_A: now reaches U1.4 (2_OUT2)
- net MG_A: now also J3.3 (Pin_3), R7.1
- net SDA: now reaches U1.40 (18_A4_SDA)
- net SDA: now also J5.3 (Pin_3), J6.3 (Pin_3)
- net SCL: now reaches U1.41 (19_A5_SCL)
- net SCL: now also J5.2 (Pin_2), J6.2 (Pin_2)
- net at U1.42 (20_A6_TX5_LRCLK1): now also R2.1, R5.1
- net at U1.43 (21_A7_RX5_BCLK1): now also R1.1, R4.1
- net at U1.48 (VIN): now also C1.1, C2.1, D1.1 (K), D2.1 (K)
- net MG_B: now reaches U1.5 (3_LRCLK2)
- net MG_B: now also J3.4 (Pin_4), R8.1
- net at U1.7 (5_IN2): now also R9.1
- net at U1.8 (6_OUT1D): now also R3.1
- new net +5V: D1.2 (A), J1.1 (Pin_1)
- new net BCLK_I: J2.2 (Pin_2), R1.2
- new net BCLK_O: J4.2 (Pin_2), R4.2
- new net CLIP: J9.2 (Pin_2), R14.2
- new net DATA_I: J2.1 (Pin_1), R3.2
- new net DATA_O: J4.1 (Pin_1), R9.2
- new net LRCLK_I: J2.3 (Pin_3), R2.2
- new net LRCLK_O: J4.3 (Pin_3), R5.2

Commit message: WIP
Changed lines of the file:
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@@
-	)
-	(junction
-		(at 231.14 67.31)
-		(diameter 0)
-		(color 0 0 0 0)
 	)
 	(junction
@@
 	(wire
 		(pts
+			(xy 231.14 67.31) (xy 234.95 67.31)
+		)
+		(stroke
+			(width 0)
+			(type default)
+		)
+	)
+	(wire
+		(pts
 			(xy 140.97 64.77) (xy 199.39 64.77)
 		)
@@
 	(wire
 		(pts
-			(xy 229.87 67.31) (xy 231.14 67.31)
-		)
-		(stroke
-			(width 0)
-			(type default)
-		)
-	)
-	(wire
-		(pts
 			(xy 157.48 116.84) (xy 187.96 116.84)
 		)
@@
 		)
 		(stroke
-			(width 0)
-			(type default)
-		)
-	)
-	(wire
-		(pts
-			(xy 231.14 67.31) (xy 234.95 67.31)
-		)
-		(stroke

Commit message: WIP
Connections:
- net GND: now also J3.4 (Pin_4), J8.4 (Pin_4); no longer J3.1 (Pin_1), J8.1 (Pin_1)
- net MGBTN: now also J3.3 (Pin_3); no longer J3.2 (Pin_2)
- net MG_A: now also J3.2 (Pin_2); no longer J3.3 (Pin_3)
- net MG_B: now also J3.1 (Pin_1); no longer J3.4 (Pin_4)
- net SPBTN: now also J8.3 (Pin_3); no longer J8.2 (Pin_2)
- net SP_A: now also J8.2 (Pin_2); no longer J8.3 (Pin_3)
- net SP_B: now also J8.1 (Pin_1); no longer J8.4 (Pin_4)
Changed lines of the file:
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@@
 	(symbol
 		(lib_id "Connector:Conn_01x04_Pin")
-		(at 21.59 88.9 0)
-		(unit 1)
-		(exclude_from_sim no)
-		(in_bom yes)
-		(on_board yes)
-		(dnp no)
-		(fields_autoplaced yes)
+		(at 21.59 91.44 0)
+		(mirror x)
+		(unit 1)
+		(exclude_from_sim no)
+		(in_bom yes)
+		(on_board yes)
+		(dnp no)
 		(property "Reference" "J8"
-			(at 22.225 81.28 0)
+			(at 22.86 84.074 0)
 			(effects
 				(font
@@
 		)
 		(property "Value" "SPARE"
-			(at 22.225 83.82 0)
+			(at 23.114 81.534 0)
 			(effects
 				(font
@@
 		)
 		(property "Footprint" "Connector_JST:JST_PH_B4B-PH-K_1x04_P2.00mm_Vertical"
-			(at 21.59 88.9 0)
-			(effects
-				(font
-					(size 1.27 1.27)
-				)
-				(hide yes)
-			)
-		)
-		(property "Datasheet" "~"
-			(at 21.59 88.9 0)
+			(at 21.59 91.44 0)
+			(effects
+				(font
+					(size 1.27 1.27)
+				)
+				(hide yes)
+			)
+		)
+		(property "Datasheet" "~"
+			(at 21.59 91.44 0)
 			(effects
 				(font
@@
 		)
 		(property "Description" "Generic connector, single row, 01x04, script generated"
-			(at 21.59 88.9 0)
+			(at 21.59 91.44 0)
 			(effects
 				(font
@@
 	(symbol
 		(lib_id "Connector:Conn_01x04_Pin")
-		(at 26.67 62.23 0)
-		(unit 1)
-		(exclude_from_sim no)
-		(in_bom yes)
-		(on_board yes)
-		(dnp no)
-		(fields_autoplaced yes)
+		(at 26.67 64.77 0)
+		(mirror x)
+		(unit 1)
+		(exclude_from_sim no)
+		(in_bom yes)
+		(on_board yes)
+		(dnp no)
 		(property "Reference" "J3"
-			(at 27.305 54.61 0)
+			(at 28.956 56.896 0)
 			(effects
 				(font
@@
 		)
 		(property "Value" "MGAIN"
-			(at 27.305 57.15 0)
+			(at 28.956 54.356 0)
 			(effects
 				(font
@@
 		)
 		(property "Footprint" "Connector_JST:JST_PH_B4B-PH-K_1x04_P2.00mm_Vertical"
-			(at 26.67 62.23 0)
-			(effects
-				(font
-					(size 1.27 1.27)
-				)
-				(hide yes)
-			)
-		)
-		(property "Datasheet" "~"
-			(at 26.67 62.23 0)
+			(at 26.67 64.77 0)
+			(effects
+				(font
+					(size 1.27 1.27)
+				)
+				(hide yes)
+			)
+		)
+		(property "Datasheet" "~"
+			(at 26.67 64.77 0)
 			(effects
 				(font
@@
 		)
 		(property "Description" "Generic connector, single row, 01x04, script generated"
-			(at 26.67 62.23 0)
-			(effects
-				(font
+			(at 26.67 64.77 0)
+			(effects
+				(font
