File: kicad/regulator/regulator.kicad_pcb (KiCad board)
At the start: 2 copper layers, 56.5 x 47.2 mm, 32 parts, among them J1 5V Analog, J2 +-15V, J3 5V Digital, J4 AC, U1 LM317_TO-220, U2 R-78C5.0-1.0, U3 LM317_TO-220, U4 LM337_TO220

Commit message: WIP
Connections:
- C1 pad 1: Net-(J1-Pin_2) -> Net-(J1-Pin_1)
- C2 pad 1: Net-(J3-Pin_2) -> Net-(J3-Pin_1)
- J1 pad 1: GND -> Net-(J1-Pin_1)
- J1 pad 2: Net-(J1-Pin_2) -> GND
- J3 pad 1: GND -> Net-(J3-Pin_1)
- J3 pad 2: Net-(J3-Pin_2) -> GND
- R1 pad 1: Net-(J1-Pin_2) -> Net-(J1-Pin_1)
- U1 pad 2: Net-(J1-Pin_2) -> Net-(J1-Pin_1)
- U2 pad 3: Net-(J3-Pin_2) -> Net-(J3-Pin_1)
Routing:
- net Net-(J3-Pin_1): track 0.00 -> 21.3 mm
- net Net-(J1-Pin_1): track 0.00 -> 21.3 mm
- net Net-(J3-Pin_2): track 20.5 -> 0.00 mm
- net Net-(J1-Pin_2): track 20.4 -> 0.00 mm
Other:
- board text added: "+18V"
- board text added: "-18V"
- board text removed: "AC1"
- board text removed: "AC2"
- board text removed: "CT"
Changed lines of the file:
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@@
 	(net 5 "Net-(U3-ADJ)")
 	(net 6 "Net-(U4-ADJ)")
-	(net 7 "Net-(J1-Pin_2)")
-	(net 8 "Net-(J3-Pin_2)")
+	(net 7 "Net-(J1-Pin_1)")
+	(net 8 "Net-(J3-Pin_1)")
 	(net 9 "+15V")
 	(net 10 "-15V")
@@
 			(remove_unused_layers no)
 			(roundrect_rratio 0.208333)
-			(net 1 "GND")
+			(net 7 "Net-(J1-Pin_1)")
 			(pinfunction "Pin_1")
 			(pintype "passive")
@@
 			(layers "*.Cu" "*.Mask")
 			(remove_unused_layers no)
-			(net 7 "Net-(J1-Pin_2)")
+			(net 1 "GND")
 			(pinfunction "Pin_2")
 			(pintype "passive")
@@
 			(layers "*.Cu" "*.Mask")
 			(remove_unused_layers no)
-			(net 8 "Net-(J3-Pin_2)")
+			(net 8 "Net-(J3-Pin_1)")
 			(pinfunction "OUT")
 			(pintype "power_out")
@@
 			(remove_unused_layers no)
 			(roundrect_rratio 0.208333)
-			(net 7 "Net-(J1-Pin_2)")
+			(net 7 "Net-(J1-Pin_1)")
 			(pintype "passive")
 		)
@@
 			(remove_unused_layers no)
 			(roundrect_rratio 0.208333)
-			(net 1 "GND")
+			(net 8 "Net-(J3-Pin_1)")
 			(pinfunction "Pin_1")
 			(pintype "passive")
@@
 			(layers "*.Cu" "*.Mask")
 			(remove_unused_layers no)
-			(net 8 "Net-(J3-Pin_2)")
+			(net 1 "GND")
 			(pinfunction "Pin_2")
 			(pintype "passive")
@@
 			(layers "*.Cu" "*.Mask")
 			(remove_unused_layers no)
-			(net 7 "Net-(J1-Pin_2)")
+			(net 7 "Net-(J1-Pin_1)")
 			(pinfunction "VO")
 			(pintype "power_out")
@@
 			(layers "*.Cu" "*.Mask")
 			(remove_unused_layers no)
-			(net 7 "Net-(J1-Pin_2)")
+			(net 7 "Net-(J1-Pin_1)")
 			(pintype "passive")
 		)
@@
 			(remove_unused_layers no)
 			(roundrect_rratio 0.208333)
-			(net 8 "Net-(J3-Pin_2)")
+			(net 8 "Net-(J3-Pin_1)")
 			(pintype "passive")
 		)
@@
 		)
 	)
-	(gr_text "AC2"
+	(gr_text "-18V"
 		(at 53.086 73.152 0)
 		(layer "F.SilkS")
@@
 		)
 	)
-	(gr_text "AC1"
+	(gr_text "+18V"
 		(at 53.086 67.869 0)
 		(layer "F.SilkS")
@@
 		)
 	)
-	(gr_text "CT"
+	(gr_text "GND"
 		(at 52.877 70.739 0)
 		(layer "F.SilkS")
@@
 	)
 	(segment
+		(start 95.123 69.215)
+		(end 97.282 69.215)
+		(width 1)
+		(layer "F.Cu")
+		(net 7)
+	)
+	(segment
+		(start 91.821 72.517)
+		(end 95.123 69.215)
+		(width 1)
+		(layer "F.Cu")
+		(net 7)
+	)
+	(segment
 		(start 90.932 72.517)
-		(end 95.98 72.517)
+		(end 91.821 72.517)
 		(width 1)
 		(layer "F.Cu")
@@
 	)
 	(segment
-		(start 95.98 72.517)
-		(end 97.282 71.215)
-		(width 1)
-		(layer "F.Cu")
-		(net 7)
-	)
-	(segment
 		(start 85.876 80.899)
 		(end 89.813 76.962)
@@
 	)
 	(segment
-		(start 90.082401 64.77)
-		(end 90.082401 64.17)
+		(start 96.562401 57.69)
+		(end 97.282 57.69)
 		(width 1)
 		(layer "F.Cu")
@@
 	(segment
 		(start 90.082401 64.17)
-		(end 94.562401 59.69)
+		(end 96.562401 57.69)
 		(width 1)
 		(layer "F.Cu")
@@
 	)
 	(segment
-		(start 94.562401 59.69)
-		(end 97.282 59.69)
+		(start 90.082401 64.77)
+		(end 90.082401 64.17)
 		(width 1)
 		(layer "F.Cu")
