File: kicad/regulator/regulator.kicad_sch (KiCad schematic)
At the start: 30 parts, among them J1 5V Analog, J2 +-15V, J3 5V Digital, J4 AC, U1 LM317_TO-220, U2 R-78C5.0-1.0, U3 LM317_TO-220, U4 LM337_TO220

Commit message: WIP
Connections:
- net GND: now also J1.2 (Pin_2), J3.2 (Pin_2); no longer J1.1 (Pin_1), J3.1 (Pin_1)
- net at C2.1, U2.3 (OUT): now also J3.1 (Pin_1); no longer J3.2 (Pin_2)
- net at C1.1, R1.1, U1.2 (VO): now also J1.1 (Pin_1); no longer J1.2 (Pin_2)
Other:
- moved on the sheet: J1, J3
Changed lines of the file:
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@@
 	(symbol
 		(lib_id "Connector:Conn_01x02_Pin")
-		(at 254 43.18 180)
+		(at 254 40.64 0)
+		(mirror y)
 		(unit 1)
 		(exclude_from_sim no)
@@
 		(dnp no)
 		(property "Reference" "J1"
-			(at 257.048 43.18 0)
+			(at 257.048 40.64 0)
 			(effects
 				(font
@@
 		)
 		(property "Value" "5V Analog"
-			(at 261.112 40.64 0)
+			(at 261.112 43.18 0)
 			(effects
 				(font
@@
 		)
 		(property "Footprint" "Connector_JST:JST_PH_B2B-PH-K_1x02_P2.00mm_Vertical"
-			(at 254 43.18 0)
-			(effects
-				(font
-					(size 1.27 1.27)
-				)
-				(hide yes)
-			)
-		)
-		(property "Datasheet" "~"
-			(at 254 43.18 0)
+			(at 254 40.64 0)
+			(effects
+				(font
+					(size 1.27 1.27)
+				)
+				(hide yes)
+			)
+		)
+		(property "Datasheet" "~"
+			(at 254 40.64 0)
 			(effects
 				(font
@@
 		)
 		(property "Description" "Generic connector, single row, 01x02, script generated"
-			(at 254 43.18 0)
+			(at 254 40.64 0)
 			(effects
 				(font
@@
 		)
 		(instances
-			(project ""
+			(project "regulator"
 				(path "/134eaab6-56fa-4d9f-a2e0-332a6380bb18"
 					(reference "J1")
@@
 	(symbol
 		(lib_id "Connector:Conn_01x02_Pin")
-		(at 255.27 55.88 180)
-		(unit 1)
-		(exclude_from_sim no)
-		(in_bom yes)
-		(on_board yes)
-		(dnp no)
-		(fields_autoplaced yes)
+		(at 255.27 53.34 0)
+		(mirror y)
+		(unit 1)
+		(exclude_from_sim no)
+		(in_bom yes)
+		(on_board yes)
+		(dnp no)
 		(property "Reference" "J3"
-			(at 256.54 53.3399 0)
+			(at 256.54 55.8801 0)
 			(effects
 				(font
@@
 		)
 		(property "Value" "5V Digital"
-			(at 256.54 55.8799 0)
+			(at 256.54 53.3401 0)
 			(effects
 				(font
@@
 		)
 		(property "Footprint" "Connector_JST:JST_PH_B2B-PH-K_1x02_P2.00mm_Vertical"
-			(at 255.27 55.88 0)
-			(effects
-				(font
-					(size 1.27 1.27)
-				)
-				(hide yes)
-			)
-		)
-		(property "Datasheet" "~"
-			(at 255.27 55.88 0)
+			(at 255.27 53.34 0)
+			(effects
+				(font
+					(size 1.27 1.27)
+				)
+				(hide yes)
+			)
+		)
+		(property "Datasheet" "~"
+			(at 255.27 53.34 0)
 			(effects
 				(font
@@
 		)
 		(property "Description" "Generic connector, single row, 01x02, script generated"
-			(at 255.27 55.88 0)
-			(effects
-				(font
+			(at 255.27 53.34 0)
+			(effects
+				(font
